File: Wii Bluetooth Module/main.brd (EAGLE design)
At the start: 17.3 x 25.4 mm, 5 parts, among them J1 USB4085-GF-A_REVA, U1 5>3V3

Commit message: eagle project updated
Parts:
- added R1, R2: 5.1k, rcl:R0805
- moved J1 0.13 mm to (8.76, 2.03)
- flipped C1 to the bottom, turned to 0 degrees
- flipped C2 to the bottom, turned to 0 degrees
- flipped U1 to the bottom
Connections:
- new net N$1: J1.B5, R2.2
- new net N$2: J1.A5, R1.2
- net GND: now also R1.1, R2.1
Routing:
- net DP: track 21.5 -> 14.0 mm
- net N$1: track 0.00 -> 6.23 mm
- net N$2: track 0.00 -> 6.11 mm
- net 3.3V: track 17.4 -> 22.3 mm, vias 0 -> 1
- net DN: track 16.5 -> 14.3 mm, vias 1 -> 0
- net GND: track 59.4 -> 60.3 mm, vias 0 -> 2
- net VCC: track 18.7 -> 18.8 mm, vias 0 -> 1
Other:
- board text added: "Wii BT USB-C v0.3 Boyo 2020"
- board text removed: "Wii BT USB-C v1 Boyo 2020"
