File: WML-C43/WML-C43-groundplanes.kicad_pcb (KiCad board)
At the start: 2 copper layers, 20 x 30 mm, 18 parts, among them J1 TYPE-C-31-M12_13, U1 USBLC6-2SC6, U2 MCP1700-3302E_SOT23, U3 WML-C43

Commit message: v0.4
-added USB data pin ESD protection
-added low pass filter to deal with noise on VCC/+5v
-fixed the slim stack connector pinout cause the 1-8 row was flipped because my brain is pepega
Routing:
- net 3.3V: track 22.8 -> 23.6 mm
- added copper zone on B.Cu, net GND
- removed copper zone on B.Cu, net (none)
Other:
- board text removed: "WML-C43 to USB-C v0.4 Nailima 2021"
