File: WML-C43/WML-C43.sch (KiCad schematic (older format))
At the start: 13 parts

Commit message: 50% done
+footprint and symbol for WML-C43 Molex Connector
+pcb
+schematic finished
Parts:
- added U3: WML-C43, Wii-BL-Lib:WML-C43, symbol Wii-BL-Lib:WML-C43
- C1, C2, C3, C4: renamed from C?; footprint (none) -> Capacitor_SMD:C_0805_2012Metric_Pad1.15x1.40mm_HandSolder
- F1: renamed from F?; footprint (none) -> Fuse:Fuse_1206_3216Metric_Pad1.42x1.75mm_HandSolder
- J1: renamed from J?; footprint acheronConnectors:TYPE-C-31-M-12 -> acheron_Connectors:TYPE-C-31-M-12
- R1, R2, R3: renamed from R?; footprint (none) -> Resistor_SMD:R_0805_2012Metric_Pad1.15x1.40mm_HandSolder
- gave numbers to parts that had none: 4
Connections:
- net 3.3V: now also U3.13 (3.3v), U3.6 (3.3v), U3.7 (3.3v)
- net D+: now also U3.11 (D+)
- net D-: now also U3.10 (D-)
- net GND: now also U3.1 (GND), U3.16 (GND), U3.8 (GND), U3.9 (GND)
- no-connect marks 2 -> 3
Other:
- moved on the sheet: C2, C3, C4, D1, D2, F1, U1, U2

Commit message: v0.4
-added USB data pin ESD protection
-added low pass filter to deal with noise on VCC/+5v
-fixed the slim stack connector pinout cause the 1-8 row was flipped because my brain is pepega
Parts:
- added C5: 10n, Capacitor_SMD:C_0805_2012Metric_Pad1.15x1.40mm_HandSolder, symbol Device:C_Small
- added C6: 100n, Capacitor_SMD:C_0805_2012Metric_Pad1.15x1.40mm_HandSolder, symbol Device:C_Small
- added C7: 10u, Capacitor_SMD:C_0805_2012Metric_Pad1.15x1.40mm_HandSolder, symbol Device:C_Small
- added FB1: Ferrite_Bead_Small, Inductor_SMD:L_0603_1608Metric_Pad1.05x0.95mm_HandSolder, symbol Device:Ferrite_Bead_Small
- D2: footprint Diode_THT:D_DO-35_SOD27_P7.62mm_Horizontal -> Diode_SMD:D_SOD-323F
Connections:
- net GND: now also C5.2, C6.2, C7.2
- net VBUS: now also C5.1, FB1.2; no longer C3.2, F1.2, U1.5 (VBUS)
- new net VFILTER: C3.2, C6.1, C7.1, F1.2, FB1.1, U1.5 (VBUS)
Changed lines of the file:
@@
 	0    1    1    0
 $EndComp
-Text GLabel 2450 1300 0    50   Input ~ 0
-VBUS
 Wire Wire Line
 	2450 1300 2550 1300
@@
 F 0 "D2" H 3250 1167 50  0000 C CNN
 F 1 "1N914" H 3250 1076 50  0000 C CNN
-F 2 "Diode_THT:D_DO-35_SOD27_P7.62mm_Horizontal" H 3250 775 50  0001 C CNN
+F 2 "Diode_SMD:D_SOD-323F" H 3250 775 50  0001 C CNN
 F 3 "http://www.vishay.com/docs/85622/1n914.pdf" H 3250 950 50  0001 C CNN
 	1    3250 950
@@
 	3050 3950 3050 3650
 Text GLabel 2900 3650 0    50   Input ~ 0
-VBUS
+VFILTER
 Wire Wire Line
 	2900 3650 3050 3650
@@
 	1    0    0    -1
 $EndComp
+Text GLabel 2450 1300 0    50   Input ~ 0
+VFILTER
+Text GLabel 4750 1500 0    50   Input ~ 0
+VBUS
+$Comp
+L Device:C_Small C5
+U 1 1 5FB59EB5
+P 5000 1600
+F 0 "C5" H 5092 1646 50  0000 L CNN
+F 1 "10n" H 5092 1555 50  0000 L CNN
+F 2 "Capacitor_SMD:C_0805_2012Metric_Pad1.15x1.40mm_HandSolder" H 5000 1600 50  0001 C CNN
+F 3 "~" H 5000 1600 50  0001 C CNN
+	1    5000 1600
+	1    0    0    -1
+$EndComp
+$Comp
+L Device:C_Small C6
+U 1 1 5FB5A6AE
+P 5550 1600
+F 0 "C6" H 5642 1646 50  0000 L CNN
+F 1 "100n" H 5642 1555 50  0000 L CNN
+F 2 "Capacitor_SMD:C_0805_2012Metric_Pad1.15x1.40mm_HandSolder" H 5550 1600 50  0001 C CNN
+F 3 "~" H 5550 1600 50  0001 C CNN
+	1    5550 1600
+	1    0    0    -1
+$EndComp
+$Comp
+L Device:Ferrite_Bead_Small FB1
+U 1 1 5FB5B2EC
+P 5250 1500
+F 0 "FB1" V 5013 1500 50  0000 C CNN
+F 1 "Ferrite_Bead_Small" V 5104 1500 50  0000 C CNN
+F 2 "Inductor_SMD:L_0603_1608Metric_Pad1.05x0.95mm_HandSolder" V 5180 1500 50  0001 C CNN
+F 3 "~" H 5250 1500 50  0001 C CNN
+	1    5250 1500
+	0    1    1    0
+$EndComp
+Wire Wire Line
+	4750 1500 5000 1500
+Wire Wire Line
+	5000 1500 5150 1500
+Connection ~ 5000 1500
+Wire Wire Line
+	5350 1500 5550 1500
+Text GLabel 6150 1500 2    50   Output ~ 0
+VFILTER
+Connection ~ 5550 1500
+Wire Wire Line
+	5000 1700 5250 1700
+$Comp
+L power:GND #PWR0108
+U 1 1 5FB62622
+P 5250 1700
+F 0 "#PWR0108" H 5250 1450 50  0001 C CNN
+F 1 "GND" H 5255 1527 50  0000 C CNN
+F 2 "" H 5250 1700 50  0001 C CNN
+F 3 "" H 5250 1700 50  0001 C CNN
+	1    5250 1700
+	1    0    0    -1
+$EndComp
+Connection ~ 5250 1700
+Wire Wire Line
+	5250 1700 5550 1700
+$Comp
+L Device:C_Small C7
+U 1 1 606AD70F
+P 5900 1600
+F 0 "C7" H 5992 1646 50  0000 L CNN
+F 1 "10u" H 5992 1555 50  0000 L CNN
+F 2 "Capacitor_SMD:C_0805_2012Metric_Pad1.15x1.40mm_HandSolder" H 5900 1600 50  0001 C CNN
+F 3 "~" H 5900 1600 50  0001 C CNN
+	1    5900 1600
+	1    0    0    -1
+$EndComp
+Wire Wire Line
+	5550 1500 5900 1500
+Wire Wire Line
+	5900 1500 6150 1500
+Connection ~ 5900 1500
+Wire Wire Line
+	5550 1700 5900 1700
+Connection ~ 5550 1700
 $EndSCHEMATC
